File: pihat-schematic-master/pihat.kicad_pcb (KiCad board)
At the start: 2 copper layers, 90.5 x 80.5 mm, 7 parts, among them J1 Raspberry_Pi_2_3, J2 2601-3114, J3 2601-3114

Commit message: Updates to Pihat
Parts:
- added J4: 5V_Connect, wago_terms:CONN5_2601-3105_WAG, F.Cu at (88.5, 113.0)
- added J5: 3V_Connect, wago_terms:CONN5_2601-3105_WAG, F.Cu at (117.0, 113.0)
- added J6: 2601-1110, wago_terms:CONN10_2601-1110_WAG, F.Cu at (93.0, 125.5)
- moved J3 41.9 mm to (90.2, 74.4), turned to 0 degrees
- moved J2 3.91 mm to (135.7, 90.4)
Routing:
- net Net-(J6-10_1): track 0.00 -> 140.1 mm
- net Net-(J5-1_1): track 0.00 -> 133.8 mm
- net Net-(J4-1_1): track 0.00 -> 89.4 mm
- net Net-(J1-GPIO14/TXD): track 0.00 -> 86.4 mm
- net Net-(J1-GPIO15/RXD): track 0.00 -> 82.8 mm
- net Net-(J1-GPIO17): track 0.00 -> 75.4 mm
- net Net-(J1-GPIO18/PWM0): track 0.00 -> 63.2 mm
- net Net-(J1-GPIO20/MOSI1): track 0.00 -> 50.0 mm
- net Net-(J1-GCLK1/GPIO5): track 0.00 -> 49.5 mm
- net Net-(J1-GPIO22): track 0.00 -> 48.3 mm
- net Net-(J1-ID_SD/GPIO0): track 0.00 -> 47.6 mm
- net Net-(J1-GPIO16): track 0.00 -> 44.4 mm
- net Net-(J1-GPIO19/MISO1): track 0.00 -> 44.2 mm
- net Net-(J1-GPIO21/SCLK1): track 0.00 -> 41.5 mm
- net Net-(J1-ID_SC/GPIO1): track 0.00 -> 39.0 mm
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Other:
- board size 90.5 x 80.5 mm -> 66.5 x 84 mm

Commit message: Began adding breakout pins
Routing:
- net Net-(J1-PWM1/GPIO13): track 23.0 -> 23.8 mm
Changed lines of the file:
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@@
 		)
 		(property "Footprint" "wago_terms:CONN5_2601-3105_WAG"
-			(at 0 0 360)
+			(at 0 0 0)
 			(layer "F.Fab")
 			(hide yes)
@@
 		)
 		(property "Datasheet" "2601-3105"
-			(at 0 0 360)
+			(at 0 0 0)
 			(layer "F.Fab")
 			(hide yes)
@@
 		)
 		(property "Description" ""
-			(at 0 0 360)
+			(at 0 0 0)
 			(layer "F.Fab")
 			(hide yes)
@@
 		)
 		(property "Footprint" "wago_terms:CONN5_2601-3105_WAG"
-			(at 0 0 360)
+			(at 0 0 0)
 			(layer "F.Fab")
 			(hide yes)
@@
 		)
 		(property "Datasheet" "2601-3105"
-			(at 0 0 360)
+			(at 0 0 0)
 			(layer "F.Fab")
 			(hide yes)
@@
 		)
 		(property "Description" ""
-			(at 0 0 360)
+			(at 0 0 0)
 			(layer "F.Fab")
 			(hide yes)
@@
 		(net 27)
 	)
+	(segment
+		(start 136.270101 75)
+		(end 135.695102 74.425001)
+		(width 0.25)
+		(layer "B.Cu")
+		(net 27)
+	)
